File: !fablabs-kicad-library.kicad_blocks/CONVERTER_USB_UART_CP2102N.kicad_block/CONVERTER_USB_UART_CP2102N.kicad_sch (KiCad schematic)
At the start: 6 parts, among them J1 USB_B_Micro, J2 UART_HEADER, U1 CP2102N-A01-GQFN28

Commit message: Fixed some bugs
Connections:
- net UART_1: now also J2.1 (Pin_1)
- net UART_2: now also J2.2 (Pin_2)
- net UART_3: now also J2.3 (Pin_3)
- net UART_4: now also J2.4 (Pin_4)
- net UART_5: now also J2.5 (Pin_5)
- net UART_6: now also J2.6 (Pin_6)
- new net: U1.29 (GND), U1.3 (GND)
Changed lines of the file:
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@@
-(kicad_sch (version 20250114) (generator "fablabs-kicad-library-builder") (generator_version "1.0.0")
+(kicad_sch (version 20260306) (generator "eeschema") (generator_version "10.0")
   (paper "A4")
   (title_block
@@
     (property "MPN" "CP2102N-A01-GQFN28" (at 30 50.24 0) (effects (font (size 1.27 1.27)) hide))
     (property "Manufacturer" "Silicon Labs" (at 30 52.78 0) (effects (font (size 1.27 1.27)) hide))
+    (instances
+      (project "fablabs"
+        (path "/2f226d8a-0ea3-44af-8b61-acd6fc20c7f6"
+          (reference "U1") (unit 1)
+        )
+      )
+    )
   )
   (symbol (lib_id "!fablabs-kicad-library:USB_B_Micro") (at 72 35 0) (unit 1) (exclude_from_sim no) (in_bom yes) (on_board yes) (dnp no)
@@
     (property "Footprint" "!fablabs-kicad-library:USB_Micro-B_Molex-105017-0001" (at 72 45.16 0) (effects (font (size 1.27 1.27)) hide))
     (property "Datasheet" "" (at 72 47.7 0) (effects (font (size 1.27 1.27)) hide))
+    (instances
+      (project "fablabs"
+        (path "/260a1342-1109-4069-b27a-9dff2e50e6a2"
+          (reference "J1") (unit 1)
+        )
+      )
+    )
   )
   (symbol (lib_id "!fablabs-kicad-library:D_TVS") (at 114 35 0) (unit 1) (exclude_from_sim no) (in_bom yes) (on_board yes) (dnp no)
@@
     (property "Footprint" "!fablabs-kicad-library:D_SOD-123" (at 114 45.16 0) (effects (font (size 1.27 1.27)) hide))
     (property "Datasheet" "" (at 114 47.7 0) (effects (font (size 1.27 1.27)) hide))
+    (instances
+      (project "fablabs"
+        (path "/012b71e1-0b2d-424f-af0f-58836e6b97b8"
+          (reference "D1") (unit 1)
+        )
+      )
+    )
   )
   (symbol (lib_id "!fablabs-kicad-library:C") (at 30 67 0) (unit 1) (exclude_from_sim no) (in_bom yes) (on_board yes) (dnp no)
@@
     (property "Footprint" "!fablabs-kicad-library:C_0603_1608Metric" (at 30 77.16 0) (effects (font (size 1.27 1.27)) hide))
     (property "Datasheet" "" (at 30 79.7 0) (effects (font (size 1.27 1.27)) hide))
+    (instances
+      (project "fablabs"
+        (path "/97458126-46bb-4768-ab6d-c7a778c902e3"
+          (reference "C1") (unit 1)
+        )
+      )
+    )
   )
   (symbol (lib_id "!fablabs-kicad-library:C") (at 72 67 0) (unit 1) (exclude_from_sim no) (in_bom yes) (on_board yes) (dnp no)
@@
     (property "Footprint" "!fablabs-kicad-library:C_0603_1608Metric" (at 72 77.16 0) (effects (font (size 1.27 1.27)) hide))
     (property "Datasheet" "" (at 72 79.7 0) (effects (font (size 1.27 1.27)) hide))
+    (instances
+      (project "fablabs"
+        (path "/01c40d07-6575-4b3c-b9b1-2bccba966ca6"
+          (reference "C2") (unit 1)
+        )
+      )
+    )
   )
   (symbol (lib_id "!fablabs-kicad-library:Conn_01x06_Pin") (at 114 67 0) (unit 1) (exclude_from_sim no) (in_bom yes) (on_board yes) (dnp no)
@@
     (property "Footprint" "!fablabs-kicad-library:PinHeader_1x06_P2.54mm_Vertical" (at 114 77.16 0) (effects (font (size 1.27 1.27)) hide))
     (property "Datasheet" "" (at 114 79.7 0) (effects (font (size 1.27 1.27)) hide))
+    (instances
+      (project "fablabs"
+        (path "/07b5e29f-128a-4932-9da8-3ef5f535df30"
+          (reference "J2") (unit 1)
+        )
+      )
+    )
   )
-  (label "UART_1" (at 119.08 72.08 0) (fields_autoplaced) (effects (font (size 1.27 1.27)) (justify left bottom)))
-  (label "UART_2" (at 119.08 69.54 0) (fields_autoplaced) (effects (font (size 1.27 1.27)) (justify left bottom)))
+  (label "UART_1" (at 119.08 61.92 0) (fields_autoplaced) (effects (font (size 1.27 1.27)) (justify left bottom)))
+  (label "UART_2" (at 119.08 64.46 0) (fields_autoplaced) (effects (font (size 1.27 1.27)) (justify left bottom)))
   (label "UART_3" (at 119.08 67 0) (fields_autoplaced) (effects (font (size 1.27 1.27)) (justify left bottom)))
-  (label "UART_4" (at 119.08 64.46 0) (fields_autoplaced) (effects (font (size 1.27 1.27)) (justify left bottom)))
-  (label "UART_5" (at 119.08 61.92 0) (fields_autoplaced) (effects (font (size 1.27 1.27)) (justify left bottom)))
-  (label "UART_6" (at 119.08 59.38 0) (fields_autoplaced) (effects (font (size 1.27 1.27)) (justify left bottom)))
+  (label "UART_4" (at 119.08 69.54 0) (fields_autoplaced) (effects (font (size 1.27 1.27)) (justify left bottom)))
+  (label "UART_5" (at 119.08 72.08 0) (fields_autoplaced) (effects (font (size 1.27 1.27)) (justify left bottom)))
+  (label "UART_6" (at 119.08 74.62 0) (fields_autoplaced) (effects (font (size 1.27 1.27)) (justify left bottom)))
+  (sheet_instances
+    (path "/" (page "1"))
+  )
 )
