File: !fablabs-kicad-library.kicad_blocks/IO_FEATHER_WING_SOCKET_SHELL.kicad_block/IO_FEATHER_WING_SOCKET_SHELL.kicad_pcb (KiCad board)
At the start: 2 copper layers, 2 parts, among them J1 FEATHER_LEFT, J2 FEATHER_RIGHT

Commit message: Fixed some bugs
Parts:
- moved J2 94.3 mm to (80.0, 50.0)
- moved J1 70.7 mm to (50.0, 50.0)
Changed lines of the file:
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@@
-(kicad_pcb (version 20240108) (generator "fablabs-kicad-library-builder") (generator_version "1.0.0")
+(kicad_pcb (version 20260206) (generator "eeschema") (generator_version "10.0")
   (general (thickness 1.6))
   (paper "A4")
@@
   	(generator "kicad-footprint-generator")
   	(layer "F.Cu")
+    (at 50 50 0)
   	(descr "Through hole straight socket strip, 1x12, 2.54mm pitch, single row (from Kicad 4.0.7), script generated")
   	(tags "Through hole socket strip THT 1x12 2.54mm single row")
   	(property "Reference" "J1"
-    (at 50 50 0)
+  		(at 0 -2.77 0)
   		(layer "F.SilkS")
   		(effects
@@
   	(generator "kicad-footprint-generator")
   	(layer "F.Cu")
+    (at 80 50 0)
   	(descr "Through hole straight socket strip, 1x16, 2.54mm pitch, single row (from Kicad 4.0.7), script generated")
   	(tags "Through hole socket strip THT 1x16 2.54mm single row")
   	(property "Reference" "J2"
-    (at 80 50 0)
-  		(layer "F.SilkS")
-  		(effects
+  		(at 0 -2.77 0)
+  		(layer "F.SilkS")
+  		(effects
