File: !fablabs-kicad-library.kicad_blocks/IO_FEATHER_WING_SOCKET_SHELL.kicad_block/IO_FEATHER_WING_SOCKET_SHELL.kicad_sch (KiCad schematic)
At the start: 2 parts, among them J1 FEATHER_LEFT, J2 FEATHER_RIGHT

Commit message: Fixed some bugs
Connections:
- net FEATHER_L_1: now also J1.1 (Pin_1)
- net FEATHER_L_10: now also J1.10 (Pin_10)
- net FEATHER_L_11: now also J1.11 (Pin_11)
- net FEATHER_L_12: now also J1.12 (Pin_12)
- net FEATHER_L_2: now also J1.2 (Pin_2)
- net FEATHER_L_3: now also J1.3 (Pin_3)
- net FEATHER_L_4: now also J1.4 (Pin_4)
- net FEATHER_L_5: now also J1.5 (Pin_5)
- net FEATHER_L_6: now also J1.6 (Pin_6)
- net FEATHER_L_7: now also J1.7 (Pin_7)
- net FEATHER_L_8: now also J1.8 (Pin_8)
- net FEATHER_L_9: now also J1.9 (Pin_9)
- net FEATHER_R_1: now also J2.1 (Pin_1)
- net FEATHER_R_10: now also J2.10 (Pin_10)
- net FEATHER_R_11: now also J2.11 (Pin_11)
- net FEATHER_R_12: now also J2.12 (Pin_12)
- net FEATHER_R_13: now also J2.13 (Pin_13)
- net FEATHER_R_14: now also J2.14 (Pin_14)
- net FEATHER_R_15: now also J2.15 (Pin_15)
- net FEATHER_R_16: now also J2.16 (Pin_16)
- net FEATHER_R_2: now also J2.2 (Pin_2)
- net FEATHER_R_3: now also J2.3 (Pin_3)
- net FEATHER_R_4: now also J2.4 (Pin_4)
- net FEATHER_R_5: now also J2.5 (Pin_5)
- net FEATHER_R_6: now also J2.6 (Pin_6)
- net FEATHER_R_7: now also J2.7 (Pin_7)
- net FEATHER_R_8: now also J2.8 (Pin_8)
- net FEATHER_R_9: now also J2.9 (Pin_9)
Changed lines of the file:
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@@
-(kicad_sch (version 20250114) (generator "fablabs-kicad-library-builder") (generator_version "1.0.0")
+(kicad_sch (version 20260306) (generator "eeschema") (generator_version "10.0")
   (paper "A4")
   (title_block
@@
     (property "Footprint" "!fablabs-kicad-library:PinSocket_1x12_P2.54mm_Vertical" (at 30 45.16 0) (effects (font (size 1.27 1.27)) hide))
     (property "Datasheet" "" (at 30 47.7 0) (effects (font (size 1.27 1.27)) hide))
+    (instances
+      (project "fablabs"
+        (path "/35fbd4df-9e23-4993-b33b-fd8e163a8f6f"
+          (reference "J1") (unit 1)
+        )
+      )
+    )
   )
-  (label "FEATHER_L_1" (at 35.08 47.7 0) (fields_autoplaced) (effects (font (size 1.27 1.27)) (justify left bottom)))
-  (label "FEATHER_L_2" (at 35.08 45.16 0) (fields_autoplaced) (effects (font (size 1.27 1.27)) (justify left bottom)))
-  (label "FEATHER_L_3" (at 35.08 42.62 0) (fields_autoplaced) (effects (font (size 1.27 1.27)) (justify left bottom)))
-  (label "FEATHER_L_4" (at 35.08 40.08 0) (fields_autoplaced) (effects (font (size 1.27 1.27)) (justify left bottom)))
-  (label "FEATHER_L_5" (at 35.08 37.54 0) (fields_autoplaced) (effects (font (size 1.27 1.27)) (justify left bottom)))
+  (label "FEATHER_L_1" (at 35.08 22.3 0) (fields_autoplaced) (effects (font (size 1.27 1.27)) (justify left bottom)))
+  (label "FEATHER_L_2" (at 35.08 24.84 0) (fields_autoplaced) (effects (font (size 1.27 1.27)) (justify left bottom)))
+  (label "FEATHER_L_3" (at 35.08 27.38 0) (fields_autoplaced) (effects (font (size 1.27 1.27)) (justify left bottom)))
+  (label "FEATHER_L_4" (at 35.08 29.92 0) (fields_autoplaced) (effects (font (size 1.27 1.27)) (justify left bottom)))
+  (label "FEATHER_L_5" (at 35.08 32.46 0) (fields_autoplaced) (effects (font (size 1.27 1.27)) (justify left bottom)))
   (label "FEATHER_L_6" (at 35.08 35 0) (fields_autoplaced) (effects (font (size 1.27 1.27)) (justify left bottom)))
-  (label "FEATHER_L_7" (at 35.08 32.46 0) (fields_autoplaced) (effects (font (size 1.27 1.27)) (justify left bottom)))
-  (label "FEATHER_L_8" (at 35.08 29.92 0) (fields_autoplaced) (effects (font (size 1.27 1.27)) (justify left bottom)))
-  (label "FEATHER_L_9" (at 35.08 27.38 0) (fields_autoplaced) (effects (font (size 1.27 1.27)) (justify left bottom)))
-  (label "FEATHER_L_10" (at 35.08 24.84 0) (fields_autoplaced) (effects (font (size 1.27 1.27)) (justify left bottom)))
-  (label "FEATHER_L_11" (at 35.08 22.3 0) (fields_autoplaced) (effects (font (size 1.27 1.27)) (justify left bottom)))
-  (label "FEATHER_L_12" (at 35.08 19.76 0) (fields_autoplaced) (effects (font (size 1.27 1.27)) (justify left bottom)))
+  (label "FEATHER_L_7" (at 35.08 37.54 0) (fields_autoplaced) (effects (font (size 1.27 1.27)) (justify left bottom)))
+  (label "FEATHER_L_8" (at 35.08 40.08 0) (fields_autoplaced) (effects (font (size 1.27 1.27)) (justify left bottom)))
+  (label "FEATHER_L_9" (at 35.08 42.62 0) (fields_autoplaced) (effects (font (size 1.27 1.27)) (justify left bottom)))
+  (label "FEATHER_L_10" (at 35.08 45.16 0) (fields_autoplaced) (effects (font (size 1.27 1.27)) (justify left bottom)))
+  (label "FEATHER_L_11" (at 35.08 47.7 0) (fields_autoplaced) (effects (font (size 1.27 1.27)) (justify left bottom)))
+  (label "FEATHER_L_12" (at 35.08 50.24 0) (fields_autoplaced) (effects (font (size 1.27 1.27)) (justify left bottom)))
   (symbol (lib_id "!fablabs-kicad-library:Conn_01x16_Pin") (at 72 35 0) (unit 1) (exclude_from_sim no) (in_bom yes) (on_board yes) (dnp no)
     (property "Reference" "J2" (at 72 27.38 0) (effects (font (size 1.27 1.27))))
@@
     (property "Footprint" "!fablabs-kicad-library:PinSocket_1x16_P2.54mm_Vertical" (at 72 45.16 0) (effects (font (size 1.27 1.27)) hide))
     (property "Datasheet" "" (at 72 47.7 0) (effects (font (size 1.27 1.27)) hide))
+    (instances
+      (project "fablabs"
+        (path "/9137d555-9673-40c6-9176-0ccd9d04dd07"
+          (reference "J2") (unit 1)
+        )
+      )
+    )
   )
-  (label "FEATHER_R_1" (at 77.08 52.78 0) (fields_autoplaced) (effects (font (size 1.27 1.27)) (justify left bottom)))
-  (label "FEATHER_R_2" (at 77.08 50.24 0) (fields_autoplaced) (effects (font (size 1.27 1.27)) (justify left bottom)))
-  (label "FEATHER_R_3" (at 77.08 47.7 0) (fields_autoplaced) (effects (font (size 1.27 1.27)) (justify left bottom)))
-  (label "FEATHER_R_4" (at 77.08 45.16 0) (fields_autoplaced) (effects (font (size 1.27 1.27)) (justify left bottom)))
-  (label "FEATHER_R_5" (at 77.08 42.62 0) (fields_autoplaced) (effects (font (size 1.27 1.27)) (justify left bottom)))
-  (label "FEATHER_R_6" (at 77.08 40.08 0) (fields_autoplaced) (effects (font (size 1.27 1.27)) (justify left bottom)))
-  (label "FEATHER_R_7" (at 77.08 37.54 0) (fields_autoplaced) (effects (font (size 1.27 1.27)) (justify left bottom)))
+  (label "FEATHER_R_1" (at 77.08 17.22 0) (fields_autoplaced) (effects (font (size 1.27 1.27)) (justify left bottom)))
+  (label "FEATHER_R_2" (at 77.08 19.76 0) (fields_autoplaced) (effects (font (size 1.27 1.27)) (justify left bottom)))
+  (label "FEATHER_R_3" (at 77.08 22.3 0) (fields_autoplaced) (effects (font (size 1.27 1.27)) (justify left bottom)))
+  (label "FEATHER_R_4" (at 77.08 24.84 0) (fields_autoplaced) (effects (font (size 1.27 1.27)) (justify left bottom)))
+  (label "FEATHER_R_5" (at 77.08 27.38 0) (fields_autoplaced) (effects (font (size 1.27 1.27)) (justify left bottom)))
+  (label "FEATHER_R_6" (at 77.08 29.92 0) (fields_autoplaced) (effects (font (size 1.27 1.27)) (justify left bottom)))
+  (label "FEATHER_R_7" (at 77.08 32.46 0) (fields_autoplaced) (effects (font (size 1.27 1.27)) (justify left bottom)))
   (label "FEATHER_R_8" (at 77.08 35 0) (fields_autoplaced) (effects (font (size 1.27 1.27)) (justify left bottom)))
-  (label "FEATHER_R_9" (at 77.08 32.46 0) (fields_autoplaced) (effects (font (size 1.27 1.27)) (justify left bottom)))
-  (label "FEATHER_R_10" (at 77.08 29.92 0) (fields_autoplaced) (effects (font (size 1.27 1.27)) (justify left bottom)))
-  (label "FEATHER_R_11" (at 77.08 27.38 0) (fields_autoplaced) (effects (font (size 1.27 1.27)) (justify left bottom)))
-  (label "FEATHER_R_12" (at 77.08 24.84 0) (fields_autoplaced) (effects (font (size 1.27 1.27)) (justify left bottom)))
-  (label "FEATHER_R_13" (at 77.08 22.3 0) (fields_autoplaced) (effects (font (size 1.27 1.27)) (justify left bottom)))
-  (label "FEATHER_R_14" (at 77.08 19.76 0) (fields_autoplaced) (effects (font (size 1.27 1.27)) (justify left bottom)))
-  (label "FEATHER_R_15" (at 77.08 17.22 0) (fields_autoplaced) (effects (font (size 1.27 1.27)) (justify left bottom)))
-  (label "FEATHER_R_16" (at 77.08 14.68 0) (fields_autoplaced) (effects (font (size 1.27 1.27)) (justify left bottom)))
+  (label "FEATHER_R_9" (at 77.08 37.54 0) (fields_autoplaced) (effects (font (size 1.27 1.27)) (justify left bottom)))
+  (label "FEATHER_R_10" (at 77.08 40.08 0) (fields_autoplaced) (effects (font (size 1.27 1.27)) (justify left bottom)))
+  (label "FEATHER_R_11" (at 77.08 42.62 0) (fields_autoplaced) (effects (font (size 1.27 1.27)) (justify left bottom)))
+  (label "FEATHER_R_12" (at 77.08 45.16 0) (fields_autoplaced) (effects (font (size 1.27 1.27)) (justify left bottom)))
+  (label "FEATHER_R_13" (at 77.08 47.7 0) (fields_autoplaced) (effects (font (size 1.27 1.27)) (justify left bottom)))
+  (label "FEATHER_R_14" (at 77.08 50.24 0) (fields_autoplaced) (effects (font (size 1.27 1.27)) (justify left bottom)))
+  (label "FEATHER_R_15" (at 77.08 52.78 0) (fields_autoplaced) (effects (font (size 1.27 1.27)) (justify left bottom)))
+  (label "FEATHER_R_16" (at 77.08 55.32 0) (fields_autoplaced) (effects (font (size 1.27 1.27)) (justify left bottom)))
+  (sheet_instances
+    (path "/" (page "1"))
+  )
 )
