File: !fablabs-kicad-library.kicad_blocks/IO_LED_STATUS_TRIPLE.kicad_block/IO_LED_STATUS_TRIPLE.kicad_sch (KiCad schematic)
At the start: 7 parts, among them J1 LED_CTRL

Commit message: Fixed some bugs
Connections:
- net GND: now also R1.2, R2.2, R3.2
- net LED_ACT_A: now also D2.1 (K)
- net LED_ACT_K: now also D2.2 (A), R2.1
- net LED_CTRL_1: now also J1.1 (Pin_1)
- net LED_CTRL_2: now also J1.2 (Pin_2)
- net LED_CTRL_3: now also J1.3 (Pin_3)
- net LED_CTRL_4: now also J1.4 (Pin_4)
- net LED_FAULT_A: now also D3.1 (K)
- net LED_FAULT_K: now also D3.2 (A), R3.1
- net LED_PWR_A: now also D1.1 (K)
- net LED_PWR_K: now also D1.2 (A), R1.1
Changed lines of the file:
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@@
-(kicad_sch (version 20250114) (generator "fablabs-kicad-library-builder") (generator_version "1.0.0")
+(kicad_sch (version 20260306) (generator "eeschema") (generator_version "10.0")
   (paper "A4")
   (title_block
@@
     (property "Footprint" "!fablabs-kicad-library:LED_0603_1608Metric" (at 30 45.16 0) (effects (font (size 1.27 1.27)) hide))
     (property "Datasheet" "" (at 30 47.7 0) (effects (font (size 1.27 1.27)) hide))
+    (instances
+      (project "fablabs"
+        (path "/2d4bea46-7cb6-4e51-92f9-c866f49924a7"
+          (reference "D1") (unit 1)
+        )
+      )
+    )
   )
   (label "LED_PWR_A" (at 26.19 35 0) (fields_autoplaced) (effects (font (size 1.27 1.27)) (justify left bottom)))
@@
     (property "Footprint" "!fablabs-kicad-library:R_0603_1608Metric" (at 72 45.16 0) (effects (font (size 1.27 1.27)) hide))
     (property "Datasheet" "" (at 72 47.7 0) (effects (font (size 1.27 1.27)) hide))
+    (instances
+      (project "fablabs"
+        (path "/fb637183-c479-40a0-9f5f-37c71060afe0"
+          (reference "R1") (unit 1)
+        )
+      )
+    )
   )
-  (label "LED_PWR_K" (at 72 38.81 0) (fields_autoplaced) (effects (font (size 1.27 1.27)) (justify left bottom)))
-  (label "GND" (at 72 31.19 0) (fields_autoplaced) (effects (font (size 1.27 1.27)) (justify left bottom)))
+  (label "LED_PWR_K" (at 72 31.19 0) (fields_autoplaced) (effects (font (size 1.27 1.27)) (justify left bottom)))
+  (label "GND" (at 72 38.81 0) (fields_autoplaced) (effects (font (size 1.27 1.27)) (justify left bottom)))
   (symbol (lib_id "!fablabs-kicad-library:LED") (at 114 35 0) (unit 1) (exclude_from_sim no) (in_bom yes) (on_board yes) (dnp no)
     (property "Reference" "D2" (at 114 27.38 0) (effects (font (size 1.27 1.27))))
@@
     (property "Footprint" "!fablabs-kicad-library:LED_0603_1608Metric" (at 114 45.16 0) (effects (font (size 1.27 1.27)) hide))
     (property "Datasheet" "" (at 114 47.7 0) (effects (font (size 1.27 1.27)) hide))
+    (instances
+      (project "fablabs"
+        (path "/92c58539-5603-4c99-bf33-b70eff266647"
+          (reference "D2") (unit 1)
+        )
+      )
+    )
   )
   (label "LED_ACT_A" (at 110.19 35 0) (fields_autoplaced) (effects (font (size 1.27 1.27)) (justify left bottom)))
@@
     (property "Footprint" "!fablabs-kicad-library:R_0603_1608Metric" (at 30 77.16 0) (effects (font (size 1.27 1.27)) hide))
     (property "Datasheet" "" (at 30 79.7 0) (effects (font (size 1.27 1.27)) hide))
+    (instances
+      (project "fablabs"
+        (path "/d5978442-0f0d-466f-b809-92eb7378c99b"
+          (reference "R2") (unit 1)
+        )
+      )
+    )
   )
-  (label "LED_ACT_K" (at 30 70.81 0) (fields_autoplaced) (effects (font (size 1.27 1.27)) (justify left bottom)))
-  (label "GND" (at 30 63.19 0) (fields_autoplaced) (effects (font (size 1.27 1.27)) (justify left bottom)))
+  (label "LED_ACT_K" (at 30 63.19 0) (fields_autoplaced) (effects (font (size 1.27 1.27)) (justify left bottom)))
+  (label "GND" (at 30 70.81 0) (fields_autoplaced) (effects (font (size 1.27 1.27)) (justify left bottom)))
   (symbol (lib_id "!fablabs-kicad-library:LED") (at 72 67 0) (unit 1) (exclude_from_sim no) (in_bom yes) (on_board yes) (dnp no)
     (property "Reference" "D3" (at 72 59.38 0) (effects (font (size 1.27 1.27))))
@@
     (property "Footprint" "!fablabs-kicad-library:LED_0603_1608Metric" (at 72 77.16 0) (effects (font (size 1.27 1.27)) hide))
     (property "Datasheet" "" (at 72 79.7 0) (effects (font (size 1.27 1.27)) hide))
+    (instances
+      (project "fablabs"
+        (path "/a9f598be-38fd-4885-85c5-e835f664e0a7"
+          (reference "D3") (unit 1)
+        )
+      )
+    )
   )
   (label "LED_FAULT_A" (at 68.19 67 0) (fields_autoplaced) (effects (font (size 1.27 1.27)) (justify left bottom)))
@@
     (property "Footprint" "!fablabs-kicad-library:R_0603_1608Metric" (at 114 77.16 0) (effects (font (size 1.27 1.27)) hide))
     (property "Datasheet" "" (at 114 79.7 0) (effects (font (size 1.27 1.27)) hide))
+    (instances
+      (project "fablabs"
+        (path "/437fb34d-2910-4b37-b5de-f9a3be5aac93"
+          (reference "R3") (unit 1)
+        )
+      )
+    )
   )
-  (label "LED_FAULT_K" (at 114 70.81 0) (fields_autoplaced) (effects (font (size 1.27 1.27)) (justify left bottom)))
-  (label "GND" (at 114 63.19 0) (fields_autoplaced) (effects (font (size 1.27 1.27)) (justify left bottom)))
+  (label "LED_FAULT_K" (at 114 63.19 0) (fields_autoplaced) (effects (font (size 1.27 1.27)) (justify left bottom)))
+  (label "GND" (at 114 70.81 0) (fields_autoplaced) (effects (font (size 1.27 1.27)) (justify left bottom)))
   (symbol (lib_id "!fablabs-kicad-library:Conn_01x04_Pin") (at 30 99 0) (unit 1) (exclude_from_sim no) (in_bom yes) (on_board yes) (dnp no)
     (property "Reference" "J1" (at 30 91.38 0) (effects (font (size 1.27 1.27))))
@@
     (property "Footprint" "!fablabs-kicad-library:PinHeader_1x04_P2.54mm_Vertical" (at 30 109.16 0) (effects (font (size 1.27 1.27)) hide))
     (property "Datasheet" "" (at 30 111.7 0) (effects (font (size 1.27 1.27)) hide))
+    (instances
+      (project "fablabs"
+        (path "/c4f95b37-9ea4-447c-9c1d-1c4b05eba08e"
+          (reference "J1") (unit 1)
+        )
+      )
+    )
   )
-  (label "LED_CTRL_1" (at 35.08 101.54 0) (fields_autoplaced) (effects (font (size 1.27 1.27)) (justify left bottom)))
+  (label "LED_CTRL_1" (at 35.08 96.46 0) (fields_autoplaced) (effects (font (size 1.27 1.27)) (justify left bottom)))
   (label "LED_CTRL_2" (at 35.08 99 0) (fields_autoplaced) (effects (font (size 1.27 1.27)) (justify left bottom)))
-  (label "LED_CTRL_3" (at 35.08 96.46 0) (fields_autoplaced) (effects (font (size 1.27 1.27)) (justify left bottom)))
-  (label "LED_CTRL_4" (at 35.08 93.92 0) (fields_autoplaced) (effects (font (size 1.27 1.27)) (justify left bottom)))
+  (label "LED_CTRL_3" (at 35.08 101.54 0) (fields_autoplaced) (effects (font (size 1.27 1.27)) (justify left bottom)))
+  (label "LED_CTRL_4" (at 35.08 104.08 0) (fields_autoplaced) (effects (font (size 1.27 1.27)) (justify left bottom)))
+  (sheet_instances
+    (path "/" (page "1"))
+  )
 )
