File: !fablabs-kicad-library.kicad_blocks/IO_MIKROBUS_SOCKET_SHELL.kicad_block/IO_MIKROBUS_SOCKET_SHELL.kicad_sch (KiCad schematic)
At the start: 2 parts, among them J1 MIKROBUS_LEFT, J2 MIKROBUS_RIGHT

Commit message: Fixed some bugs
Connections:
- net +3V3: now also J1.7 (Pin_7)
- net +5V: now also J2.7 (Pin_7)
- net AN: now also J1.1 (Pin_1)
- net CS: now also J1.3 (Pin_3)
- net GND: now also J1.8 (Pin_8), J2.8 (Pin_8)
- net INT: now also J2.2 (Pin_2)
- net MISO: now also J1.5 (Pin_5)
- net MOSI: now also J1.6 (Pin_6)
- net PWM: now also J2.1 (Pin_1)
- net RST: now also J1.2 (Pin_2)
- net RX: now also J2.3 (Pin_3)
- net SCK: now also J1.4 (Pin_4)
- net SCL: now also J2.5 (Pin_5)
- net SDA: now also J2.6 (Pin_6)
- net TX: now also J2.4 (Pin_4)
Changed lines of the file:
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@@
-(kicad_sch (version 20250114) (generator "fablabs-kicad-library-builder") (generator_version "1.0.0")
+(kicad_sch (version 20260306) (generator "eeschema") (generator_version "10.0")
   (paper "A4")
   (title_block
@@
     (property "Footprint" "!fablabs-kicad-library:PinSocket_1x08_P2.54mm_Vertical" (at 30 45.16 0) (effects (font (size 1.27 1.27)) hide))
     (property "Datasheet" "" (at 30 47.7 0) (effects (font (size 1.27 1.27)) hide))
+    (instances
+      (project "fablabs"
+        (path "/51d74b2b-5039-4bd5-8cdf-f1c8f8416177"
+          (reference "J1") (unit 1)
+        )
+      )
+    )
   )
-  (label "AN" (at 35.08 42.62 0) (fields_autoplaced) (effects (font (size 1.27 1.27)) (justify left bottom)))
-  (label "RST" (at 35.08 40.08 0) (fields_autoplaced) (effects (font (size 1.27 1.27)) (justify left bottom)))
-  (label "CS" (at 35.08 37.54 0) (fields_autoplaced) (effects (font (size 1.27 1.27)) (justify left bottom)))
+  (label "AN" (at 35.08 27.38 0) (fields_autoplaced) (effects (font (size 1.27 1.27)) (justify left bottom)))
+  (label "RST" (at 35.08 29.92 0) (fields_autoplaced) (effects (font (size 1.27 1.27)) (justify left bottom)))
+  (label "CS" (at 35.08 32.46 0) (fields_autoplaced) (effects (font (size 1.27 1.27)) (justify left bottom)))
   (label "SCK" (at 35.08 35 0) (fields_autoplaced) (effects (font (size 1.27 1.27)) (justify left bottom)))
-  (label "MISO" (at 35.08 32.46 0) (fields_autoplaced) (effects (font (size 1.27 1.27)) (justify left bottom)))
-  (label "MOSI" (at 35.08 29.92 0) (fields_autoplaced) (effects (font (size 1.27 1.27)) (justify left bottom)))
-  (label "+3V3" (at 35.08 27.38 0) (fields_autoplaced) (effects (font (size 1.27 1.27)) (justify left bottom)))
-  (label "GND" (at 35.08 24.84 0) (fields_autoplaced) (effects (font (size 1.27 1.27)) (justify left bottom)))
+  (label "MISO" (at 35.08 37.54 0) (fields_autoplaced) (effects (font (size 1.27 1.27)) (justify left bottom)))
+  (label "MOSI" (at 35.08 40.08 0) (fields_autoplaced) (effects (font (size 1.27 1.27)) (justify left bottom)))
+  (label "+3V3" (at 35.08 42.62 0) (fields_autoplaced) (effects (font (size 1.27 1.27)) (justify left bottom)))
+  (label "GND" (at 35.08 45.16 0) (fields_autoplaced) (effects (font (size 1.27 1.27)) (justify left bottom)))
   (symbol (lib_id "!fablabs-kicad-library:Conn_01x08_Pin") (at 72 35 0) (unit 1) (exclude_from_sim no) (in_bom yes) (on_board yes) (dnp no)
     (property "Reference" "J2" (at 72 27.38 0) (effects (font (size 1.27 1.27))))
@@
     (property "Footprint" "!fablabs-kicad-library:PinSocket_1x08_P2.54mm_Vertical" (at 72 45.16 0) (effects (font (size 1.27 1.27)) hide))
     (property "Datasheet" "" (at 72 47.7 0) (effects (font (size 1.27 1.27)) hide))
+    (instances
+      (project "fablabs"
+        (path "/7229c1f1-7fe0-408c-adc0-38e82767bd0d"
+          (reference "J2") (unit 1)
+        )
+      )
+    )
   )
-  (label "PWM" (at 77.08 42.62 0) (fields_autoplaced) (effects (font (size 1.27 1.27)) (justify left bottom)))
-  (label "INT" (at 77.08 40.08 0) (fields_autoplaced) (effects (font (size 1.27 1.27)) (justify left bottom)))
-  (label "RX" (at 77.08 37.54 0) (fields_autoplaced) (effects (font (size 1.27 1.27)) (justify left bottom)))
+  (label "PWM" (at 77.08 27.38 0) (fields_autoplaced) (effects (font (size 1.27 1.27)) (justify left bottom)))
+  (label "INT" (at 77.08 29.92 0) (fields_autoplaced) (effects (font (size 1.27 1.27)) (justify left bottom)))
+  (label "RX" (at 77.08 32.46 0) (fields_autoplaced) (effects (font (size 1.27 1.27)) (justify left bottom)))
   (label "TX" (at 77.08 35 0) (fields_autoplaced) (effects (font (size 1.27 1.27)) (justify left bottom)))
-  (label "SCL" (at 77.08 32.46 0) (fields_autoplaced) (effects (font (size 1.27 1.27)) (justify left bottom)))
-  (label "SDA" (at 77.08 29.92 0) (fields_autoplaced) (effects (font (size 1.27 1.27)) (justify left bottom)))
-  (label "+5V" (at 77.08 27.38 0) (fields_autoplaced) (effects (font (size 1.27 1.27)) (justify left bottom)))
-  (label "GND" (at 77.08 24.84 0) (fields_autoplaced) (effects (font (size 1.27 1.27)) (justify left bottom)))
+  (label "SCL" (at 77.08 37.54 0) (fields_autoplaced) (effects (font (size 1.27 1.27)) (justify left bottom)))
+  (label "SDA" (at 77.08 40.08 0) (fields_autoplaced) (effects (font (size 1.27 1.27)) (justify left bottom)))
+  (label "+5V" (at 77.08 42.62 0) (fields_autoplaced) (effects (font (size 1.27 1.27)) (justify left bottom)))
+  (label "GND" (at 77.08 45.16 0) (fields_autoplaced) (effects (font (size 1.27 1.27)) (justify left bottom)))
+  (sheet_instances
+    (path "/" (page "1"))
+  )
 )
