File: !fablabs-kicad-library.kicad_blocks/MCU_ATMEGA328P_AU_MINIMUM.kicad_block/MCU_ATMEGA328P_AU_MINIMUM.kicad_sch (KiCad schematic)
At the start: 9 parts, among them J1 AVR_ISP_6, J2 ATMEGA_IO_A, J3 ATMEGA_IO_B, U1 ATmega328P-AU, Y1 16MHz

Commit message: Fixed some bugs
Connections:
- net ATMEGA_A_1: now also J2.1 (Pin_1)
- net ATMEGA_A_10: now also J2.10 (Pin_10)
- net ATMEGA_A_2: now also J2.2 (Pin_2)
- net ATMEGA_A_3: now also J2.3 (Pin_3)
- net ATMEGA_A_4: now also J2.4 (Pin_4)
- net ATMEGA_A_5: now also J2.5 (Pin_5)
- net ATMEGA_A_6: now also J2.6 (Pin_6)
- net ATMEGA_A_7: now also J2.7 (Pin_7)
- net ATMEGA_A_8: now also J2.8 (Pin_8)
- net ATMEGA_A_9: now also J2.9 (Pin_9)
- net ATMEGA_B_1: now also J3.1 (Pin_1)
- net ATMEGA_B_10: now also J3.10 (Pin_10)
- net ATMEGA_B_2: now also J3.2 (Pin_2)
- net ATMEGA_B_3: now also J3.3 (Pin_3)
- net ATMEGA_B_4: now also J3.4 (Pin_4)
- net ATMEGA_B_5: now also J3.5 (Pin_5)
- net ATMEGA_B_6: now also J3.6 (Pin_6)
- net ATMEGA_B_7: now also J3.7 (Pin_7)
- net ATMEGA_B_8: now also J3.8 (Pin_8)
- net ATMEGA_B_9: now also J3.9 (Pin_9)
- net GND: now also C3.2, J1.6 (Pin_6)
- net MISO: now also J1.1 (Pin_1)
- net MOSI: now also J1.4 (Pin_4)
- net RESET: now also J1.5 (Pin_5), R1.1
- net SCK: now also J1.3 (Pin_3)
- net VCC: now also C3.1, J1.2 (Pin_2), R1.2
