File: !fablabs-kicad-library.kicad_blocks/MCU_HEADER_ONLY_GENERIC_40PIN.kicad_block/MCU_HEADER_ONLY_GENERIC_40PIN.kicad_pcb (KiCad board)
At the start: 2 copper layers, 4 parts, among them J1 MCU_MODULE_A, J2 MCU_MODULE_B

Commit message: Fixed some bugs
Parts:
- moved C2 148.7 mm to (140.0, 50.0)
- moved C1 120.8 mm to (110.0, 50.0)
- moved J2 94.3 mm to (80.0, 50.0)
- moved J1 70.7 mm to (50.0, 50.0)
Changed lines of the file:
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@@
-(kicad_pcb (version 20240108) (generator "fablabs-kicad-library-builder") (generator_version "1.0.0")
+(kicad_pcb (version 20260206) (generator "eeschema") (generator_version "10.0")
   (general (thickness 1.6))
   (paper "A4")
@@
   	(generator "kicad-footprint-generator")
   	(layer "F.Cu")
+    (at 50 50 0)
   	(descr "Through hole straight pin header, 1x20, 2.54mm pitch, single row")
   	(tags "Through hole pin header THT 1x20 2.54mm single row")
   	(property "Reference" "J1"
-    (at 50 50 0)
+  		(at 0 -2.38 0)
   		(layer "F.SilkS")
   		(effects
@@
   	(generator "kicad-footprint-generator")
   	(layer "F.Cu")
+    (at 80 50 0)
   	(descr "Through hole straight pin header, 1x20, 2.54mm pitch, single row")
   	(tags "Through hole pin header THT 1x20 2.54mm single row")
   	(property "Reference" "J2"
-    (at 80 50 0)
+  		(at 0 -2.38 0)
   		(layer "F.SilkS")
   		(effects
@@
   	(generator "kicad-footprint-generator")
   	(layer "F.Cu")
+    (at 110 50 0)
   	(descr "Capacitor SMD 0603 (1608 Metric), square (rectangular) end terminal, IPC-7351 nominal, (Body size source: IPC-SM-782 page 76, https://www.pcb-3d.com/wordpress/wp-content/uploads/ipc-sm-782a_amendment_1_and_2.pdf)")
   	(tags "capacitor")
   	(property "Reference" "C1"
-    (at 110 50 0)
+  		(at 0 -1.43 0)
   		(layer "F.SilkS")
   		(effects
@@
   	(generator "kicad-footprint-generator")
   	(layer "F.Cu")
+    (at 140 50 0)
   	(descr "Capacitor SMD 0805 (2012 Metric), square (rectangular) end terminal, IPC-7351 nominal, (Body size source: IPC-SM-782 page 76, https://www.pcb-3d.com/wordpress/wp-content/uploads/ipc-sm-782a_amendment_1_and_2.pdf, https://docs.google.com/spreadsheets/d/1BsfQQcO9C6DZCsRaXUlFlo91Tg2WpOkGARC1WS5S8t0/edit?usp=sharing)")
   	(tags "capacitor")
   	(property "Reference" "C2"
-    (at 140 50 0)
-  		(layer "F.SilkS")
-  		(effects
+  		(at 0 -1.68 0)
+  		(layer "F.SilkS")
+  		(effects
