File: !fablabs-kicad-library.kicad_blocks/MCU_HEADER_ONLY_GENERIC_40PIN.kicad_block/MCU_HEADER_ONLY_GENERIC_40PIN.kicad_sch (KiCad schematic)
At the start: 4 parts, among them J1 MCU_MODULE_A, J2 MCU_MODULE_B

Commit message: Fixed some bugs
Connections:
- net GND: now also C1.2, C2.2
- net MCU_A_1: now also J1.1 (Pin_1)
- net MCU_A_10: now also J1.10 (Pin_10)
- net MCU_A_11: now also J1.11 (Pin_11)
- net MCU_A_12: now also J1.12 (Pin_12)
- net MCU_A_13: now also J1.13 (Pin_13)
- net MCU_A_14: now also J1.14 (Pin_14)
- net MCU_A_15: now also J1.15 (Pin_15)
- net MCU_A_16: now also J1.16 (Pin_16)
- net MCU_A_17: now also J1.17 (Pin_17)
- net MCU_A_18: now also J1.18 (Pin_18)
- net MCU_A_19: now also J1.19 (Pin_19)
- net MCU_A_2: now also J1.2 (Pin_2)
- net MCU_A_20: now also J1.20 (Pin_20)
- net MCU_A_3: now also J1.3 (Pin_3)
- net MCU_A_4: now also J1.4 (Pin_4)
- net MCU_A_5: now also J1.5 (Pin_5)
- net MCU_A_6: now also J1.6 (Pin_6)
- net MCU_A_7: now also J1.7 (Pin_7)
- net MCU_A_8: now also J1.8 (Pin_8)
- net MCU_A_9: now also J1.9 (Pin_9)
- net MCU_B_1: now also J2.1 (Pin_1)
- net MCU_B_10: now also J2.10 (Pin_10)
- net MCU_B_11: now also J2.11 (Pin_11)
- net MCU_B_12: now also J2.12 (Pin_12)
- net MCU_B_13: now also J2.13 (Pin_13)
- net MCU_B_14: now also J2.14 (Pin_14)
- net MCU_B_15: now also J2.15 (Pin_15)
- net MCU_B_16: now also J2.16 (Pin_16)
- net MCU_B_17: now also J2.17 (Pin_17)
- net MCU_B_18: now also J2.18 (Pin_18)
- net MCU_B_19: now also J2.19 (Pin_19)
- net MCU_B_2: now also J2.2 (Pin_2)
- net MCU_B_20: now also J2.20 (Pin_20)
- net MCU_B_3: now also J2.3 (Pin_3)
- net MCU_B_4: now also J2.4 (Pin_4)
- net MCU_B_5: now also J2.5 (Pin_5)
- net MCU_B_6: now also J2.6 (Pin_6)
- net MCU_B_7: now also J2.7 (Pin_7)
- net MCU_B_8: now also J2.8 (Pin_8)
- net MCU_B_9: now also J2.9 (Pin_9)
- net VCC: now also C1.1, C2.1
