File: !fablabs-kicad-library.kicad_blocks/MCU_SAMD21G18A_MINIMUM.kicad_block/MCU_SAMD21G18A_MINIMUM.kicad_pcb (KiCad board)
At the start: 2 copper layers, 9 parts, among them J1 SWD, J2 SAMD21_IO, U1 ATSAMD21G18A-AU, Y1 32.768kHz

Commit message: Fixed some bugs
Parts:
- moved C3 177.2 mm to (170.0, 50.0)
- moved J2 161.2 mm to (140.0, 80.0)
- moved C2 148.7 mm to (140.0, 50.0)
- moved J1 136.0 mm to (110.0, 80.0)
- moved C1 120.8 mm to (110.0, 50.0)
- moved R2 113.1 mm to (80.0, 80.0)
- moved R1 94.3 mm to (50.0, 80.0)
- moved Y1 94.3 mm to (80.0, 50.0)
- moved U1 70.7 mm to (50.0, 50.0)
Changed lines of the file:
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@@
-(kicad_pcb (version 20240108) (generator "fablabs-kicad-library-builder") (generator_version "1.0.0")
+(kicad_pcb (version 20260206) (generator "eeschema") (generator_version "10.0")
   (general (thickness 1.6))
   (paper "A4")
@@
   	(generator "kicad-footprint-generator")
   	(layer "F.Cu")
+    (at 50 50 0)
   	(descr "TQFP, 48 Pin (JEDEC MS-026 variation ABC, 1.00mm body thickness, https://www.jedec.org/document_search?search_api_views_fulltext=MS-026, https://ww1.microchip.com/downloads/en/PackagingSpec/00000049BZ.pdf#page=666)")
   	(tags "TQFP QFP P48GA-50-HAA-2 pkg_3304 PTQP0048KC-A C48-11 PFB0048A")
   	(property "Reference" "U1"
-    (at 50 50 0)
+  		(at 0 -5.85 0)
   		(layer "F.SilkS")
   		(effects
@@
   	)
   	(embedded_fonts no)
-  	(model "${KICAD10_3DMODEL_DIR}/Package_QFP.3dshapes/TQFP-48_7x7mm_P0.5mm.step"
+  	(model "${KIPRJMOD}/libs/!fablabs-kicad-library.3dshapes/TQFP-48_7x7mm_P0.5mm.step"
   		(offset
   			(xyz 0 0 0)
@@
   	(generator_version "10.0")
   	(layer "F.Cu")
+    (at 80 50 0)
   	(descr "SMD Crystal FC-135 https://support.epson.biz/td/api/doc_check.php?dl=brief_FC-135R_en.pdf")
   	(tags "SMD SMT Crystal")
   	(property "Reference" "Y1"
-    (at 80 50 0)
+  		(at 0 -2 0)
   		(layer "F.SilkS")
   		(effects
@@
   	(generator "kicad-footprint-generator")
   	(layer "F.Cu")
+    (at 110 50 0)
   	(descr "Capacitor SMD 0603 (1608 Metric), square (rectangular) end terminal, IPC-7351 nominal, (Body size source: IPC-SM-782 page 76, https://www.pcb-3d.com/wordpress/wp-content/uploads/ipc-sm-782a_amendment_1_and_2.pdf)")
   	(tags "capacitor")
   	(property "Reference" "C1"
-    (at 110 50 0)
+  		(at 0 -1.43 0)
   		(layer "F.SilkS")
   		(effects
@@
   	(generator "kicad-footprint-generator")
   	(layer "F.Cu")
+    (at 140 50 0)
   	(descr "Capacitor SMD 0603 (1608 Metric), square (rectangular) end terminal, IPC-7351 nominal, (Body size source: IPC-SM-782 page 76, https://www.pcb-3d.com/wordpress/wp-content/uploads/ipc-sm-782a_amendment_1_and_2.pdf)")
   	(tags "capacitor")
   	(property "Reference" "C2"
-    (at 140 50 0)
+  		(at 0 -1.43 0)
   		(layer "F.SilkS")
   		(effects
@@
   	(generator "kicad-footprint-generator")
   	(layer "F.Cu")
+    (at 170 50 0)
   	(descr "Capacitor SMD 0603 (1608 Metric), square (rectangular) end terminal, IPC-7351 nominal, (Body size source: IPC-SM-782 page 76, https://www.pcb-3d.com/wordpress/wp-content/uploads/ipc-sm-782a_amendment_1_and_2.pdf)")
   	(tags "capacitor")
   	(property "Reference" "C3"
-    (at 170 50 0)
+  		(at 0 -1.43 0)
   		(layer "F.SilkS")
   		(effects
@@
   	(generator "kicad-footprint-generator")
   	(layer "F.Cu")
+    (at 50 80 0)
   	(descr "Resistor SMD 0603 (1608 Metric), square (rectangular) end terminal, IPC-7351 nominal, (Body size source: IPC-SM-782 page 72, https://www.pcb-3d.com/wordpress/wp-content/uploads/ipc-sm-782a_amendment_1_and_2.pdf)")
   	(tags "resistor")
   	(property "Reference" "R1"
-    (at 50 80 0)
+  		(at 0 -1.43 0)
   		(layer "F.SilkS")
   		(effects
@@
   	)
   	(embedded_fonts no)
-  	(model "${KICAD10_3DMODEL_DIR}/Resistor_SMD.3dshapes/R_0603_1608Metric.step"
+  	(model "${KIPRJMOD}/libs/!fablabs-kicad-library.3dshapes/R_0603_1608Metric.step"
   		(offset
   			(xyz 0 0 0)
@@
   	(generator "kicad-footprint-generator")
   	(layer "F.Cu")
+    (at 80 80 0)
   	(descr "Resistor SMD 0603 (1608 Metric), square (rectangular) end terminal, IPC-7351 nominal, (Body size source: IPC-SM-782 page 72, https://www.pcb-3d.com/wordpress/wp-content/uploads/ipc-sm-782a_amendment_1_and_2.pdf)")
   	(tags "resistor")
   	(property "Reference" "R2"
-    (at 80 80 0)
+  		(at 0 -1.43 0)
   		(layer "F.SilkS")
   		(effects
@@
   	)
   	(embedded_fonts no)
-  	(model "${KICAD10_3DMODEL_DIR}/Resistor_SMD.3dshapes/R_0603_1608Metric.step"
+  	(model "${KIPRJMOD}/libs/!fablabs-kicad-library.3dshapes/R_0603_1608Metric.step"
   		(offset
   			(xyz 0 0 0)
@@
   	(generator "kicad-footprint-generator")
   	(layer "F.Cu")
+    (at 110 80 0)
   	(descr "Through hole straight pin header, 1x04, 2.54mm pitch, single row")
   	(tags "Through hole pin header THT 1x04 2.54mm single row")
   	(property "Reference" "J1"
-    (at 110 80 0)
+  		(at 0 -2.38 0)
   		(layer "F.SilkS")
   		(effects
@@
   	(generator "kicad-footprint-generator")
   	(layer "F.Cu")
+    (at 140 80 0)
   	(descr "Through hole straight pin header, 1x20, 2.54mm pitch, single row")
   	(tags "Through hole pin header THT 1x20 2.54mm single row")
   	(property "Reference" "J2"
-    (at 140 80 0)
-  		(layer "F.SilkS")
-  		(effects
+  		(at 0 -2.38 0)
+  		(layer "F.SilkS")
+  		(effects
