File: !fablabs-kicad-library.kicad_blocks/MCU_STM32F103C8T6_MINIMUM.kicad_block/MCU_STM32F103C8T6_MINIMUM.kicad_sch (KiCad schematic)
At the start: 10 parts, among them J1 SWD, J2 STM32_IO_A, J3 STM32_IO_B, U1 STM32F103C8Tx, Y1 8MHz

Commit message: Fixed some bugs
Connections:
- net +3V3: now also C4.1, J1.1 (Pin_1), R1.2
- net GND: now also C3.2, C4.2, J1.4 (Pin_4)
- net NRST: now also C3.1, R1.1
- net STM32_A_1: now also J2.1 (Pin_1)
- net STM32_A_10: now also J2.10 (Pin_10)
- net STM32_A_11: now also J2.11 (Pin_11)
- net STM32_A_12: now also J2.12 (Pin_12)
- net STM32_A_13: now also J2.13 (Pin_13)
- net STM32_A_14: now also J2.14 (Pin_14)
- net STM32_A_15: now also J2.15 (Pin_15)
- net STM32_A_16: now also J2.16 (Pin_16)
- net STM32_A_2: now also J2.2 (Pin_2)
- net STM32_A_3: now also J2.3 (Pin_3)
- net STM32_A_4: now also J2.4 (Pin_4)
- net STM32_A_5: now also J2.5 (Pin_5)
- net STM32_A_6: now also J2.6 (Pin_6)
- net STM32_A_7: now also J2.7 (Pin_7)
- net STM32_A_8: now also J2.8 (Pin_8)
- net STM32_A_9: now also J2.9 (Pin_9)
- net STM32_B_1: now also J3.1 (Pin_1)
- net STM32_B_10: now also J3.10 (Pin_10)
- net STM32_B_11: now also J3.11 (Pin_11)
- net STM32_B_12: now also J3.12 (Pin_12)
- net STM32_B_13: now also J3.13 (Pin_13)
- net STM32_B_14: now also J3.14 (Pin_14)
- net STM32_B_15: now also J3.15 (Pin_15)
- net STM32_B_16: now also J3.16 (Pin_16)
- net STM32_B_2: now also J3.2 (Pin_2)
- net STM32_B_3: now also J3.3 (Pin_3)
- net STM32_B_4: now also J3.4 (Pin_4)
- net STM32_B_5: now also J3.5 (Pin_5)
- net STM32_B_6: now also J3.6 (Pin_6)
- net STM32_B_7: now also J3.7 (Pin_7)
- net STM32_B_8: now also J3.8 (Pin_8)
- net STM32_B_9: now also J3.9 (Pin_9)
- net SWCLK: now also J1.3 (Pin_3)
- net SWDIO: now also J1.2 (Pin_2)
