File: !fablabs-kicad-library.kicad_blocks/POWER_BUCK_5V_LM2596S.kicad_block/POWER_BUCK_5V_LM2596S.kicad_sch (KiCad schematic)
At the start: 7 parts, among them J1 VIN, J2 5V_OUT, U1 LM2596S-5

Commit message: Fixed some bugs
Connections:
- net +5V: now also COUT1.1, L1.2
- net 5V_OUT_1: now also J2.1 (Pin_1)
- net 5V_OUT_2: now also J2.2 (Pin_2)
- net GND: now also CIN1.2, COUT1.2, D1.1 (K)
- net SW: now also D1.2 (A), L1.1
- net VIN: now also CIN1.1
- net VIN_1: now also J1.1 (Pin_1)
- net VIN_2: now also J1.2 (Pin_2)
Changed lines of the file:
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@@
-(kicad_sch (version 20250114) (generator "fablabs-kicad-library-builder") (generator_version "1.0.0")
+(kicad_sch (version 20260306) (generator "eeschema") (generator_version "10.0")
   (paper "A4")
   (title_block
@@
     (property "MPN" "LM2596S-5/NOPB" (at 30 50.24 0) (effects (font (size 1.27 1.27)) hide))
     (property "Manufacturer" "Texas Instruments" (at 30 52.78 0) (effects (font (size 1.27 1.27)) hide))
+    (instances
+      (project "fablabs"
+        (path "/5197cd51-ebae-47ce-bfbf-a4521d41d232"
+          (reference "U1") (unit 1)
+        )
+      )
+    )
   )
-  (label "VIN" (at 17.3 37.54 0) (fields_autoplaced) (effects (font (size 1.27 1.27)) (justify left bottom)))
-  (label "SW" (at 42.7 32.46 0) (fields_autoplaced) (effects (font (size 1.27 1.27)) (justify left bottom)))
-  (label "GND" (at 30 27.38 0) (fields_autoplaced) (effects (font (size 1.27 1.27)) (justify left bottom)))
-  (label "FB" (at 42.7 37.54 0) (fields_autoplaced) (effects (font (size 1.27 1.27)) (justify left bottom)))
-  (label "EN" (at 17.3 32.46 0) (fields_autoplaced) (effects (font (size 1.27 1.27)) (justify left bottom)))
+  (label "VIN" (at 17.3 32.46 0) (fields_autoplaced) (effects (font (size 1.27 1.27)) (justify left bottom)))
+  (label "SW" (at 42.7 37.54 0) (fields_autoplaced) (effects (font (size 1.27 1.27)) (justify left bottom)))
+  (label "GND" (at 30 42.62 0) (fields_autoplaced) (effects (font (size 1.27 1.27)) (justify left bottom)))
+  (label "FB" (at 42.7 32.46 0) (fields_autoplaced) (effects (font (size 1.27 1.27)) (justify left bottom)))
+  (label "EN" (at 17.3 37.54 0) (fields_autoplaced) (effects (font (size 1.27 1.27)) (justify left bottom)))
   (symbol (lib_id "!fablabs-kicad-library:D_Schottky") (at 72 35 0) (unit 1) (exclude_from_sim no) (in_bom yes) (on_board yes) (dnp no)
     (property "Reference" "D1" (at 72 27.38 0) (effects (font (size 1.27 1.27))))
@@
     (property "Footprint" "!fablabs-kicad-library:D_SOD-123" (at 72 45.16 0) (effects (font (size 1.27 1.27)) hide))
     (property "Datasheet" "" (at 72 47.7 0) (effects (font (size 1.27 1.27)) hide))
+    (instances
+      (project "fablabs"
+        (path "/3a1f9169-dc96-4cfd-a848-1946a31e23bc"
+          (reference "D1") (unit 1)
+        )
+      )
+    )
   )
   (label "GND" (at 68.19 35 0) (fields_autoplaced) (effects (font (size 1.27 1.27)) (justify left bottom)))
@@
     (property "Footprint" "!fablabs-kicad-library:L_Bourns_SRN6045TA" (at 114 45.16 0) (effects (font (size 1.27 1.27)) hide))
     (property "Datasheet" "" (at 114 47.7 0) (effects (font (size 1.27 1.27)) hide))
+    (instances
+      (project "fablabs"
+        (path "/82acd9aa-9ce5-45a5-8a2a-5e41b4e8e646"
+          (reference "L1") (unit 1)
+        )
+      )
+    )
   )
-  (label "SW" (at 114 38.81 0) (fields_autoplaced) (effects (font (size 1.27 1.27)) (justify left bottom)))
-  (label "+5V" (at 114 31.19 0) (fields_autoplaced) (effects (font (size 1.27 1.27)) (justify left bottom)))
+  (label "SW" (at 114 31.19 0) (fields_autoplaced) (effects (font (size 1.27 1.27)) (justify left bottom)))
+  (label "+5V" (at 114 38.81 0) (fields_autoplaced) (effects (font (size 1.27 1.27)) (justify left bottom)))
   (symbol (lib_id "!fablabs-kicad-library:C_Polarized") (at 30 67 0) (unit 1) (exclude_from_sim no) (in_bom yes) (on_board yes) (dnp no)
     (property "Reference" "CIN1" (at 30 59.38 0) (effects (font (size 1.27 1.27))))
@@
     (property "Footprint" "!fablabs-kicad-library:CP_Radial_D6.3mm_P2.50mm" (at 30 77.16 0) (effects (font (size 1.27 1.27)) hide))
     (property "Datasheet" "" (at 30 79.7 0) (effects (font (size 1.27 1.27)) hide))
+    (instances
+      (project "fablabs"
+        (path "/b99b99b8-afe3-433d-8229-97e6b3d0a487"
+          (reference "CIN1") (unit 1)
+        )
+      )
+    )
   )
-  (label "VIN" (at 30 70.81 0) (fields_autoplaced) (effects (font (size 1.27 1.27)) (justify left bottom)))
-  (label "GND" (at 30 63.19 0) (fields_autoplaced) (effects (font (size 1.27 1.27)) (justify left bottom)))
+  (label "VIN" (at 30 63.19 0) (fields_autoplaced) (effects (font (size 1.27 1.27)) (justify left bottom)))
+  (label "GND" (at 30 70.81 0) (fields_autoplaced) (effects (font (size 1.27 1.27)) (justify left bottom)))
   (symbol (lib_id "!fablabs-kicad-library:C_Polarized") (at 72 67 0) (unit 1) (exclude_from_sim no) (in_bom yes) (on_board yes) (dnp no)
     (property "Reference" "COUT1" (at 72 59.38 0) (effects (font (size 1.27 1.27))))
@@
     (property "Footprint" "!fablabs-kicad-library:CP_Radial_D6.3mm_P2.50mm" (at 72 77.16 0) (effects (font (size 1.27 1.27)) hide))
     (property "Datasheet" "" (at 72 79.7 0) (effects (font (size 1.27 1.27)) hide))
+    (instances
+      (project "fablabs"
+        (path "/f4f347c2-6039-4a38-ba8a-3b62f5aa7ba1"
+          (reference "COUT1") (unit 1)
+        )
+      )
+    )
   )
-  (label "+5V" (at 72 70.81 0) (fields_autoplaced) (effects (font (size 1.27 1.27)) (justify left bottom)))
-  (label "GND" (at 72 63.19 0) (fields_autoplaced) (effects (font (size 1.27 1.27)) (justify left bottom)))
+  (label "+5V" (at 72 63.19 0) (fields_autoplaced) (effects (font (size 1.27 1.27)) (justify left bottom)))
+  (label "GND" (at 72 70.81 0) (fields_autoplaced) (effects (font (size 1.27 1.27)) (justify left bottom)))
   (symbol (lib_id "!fablabs-kicad-library:Conn_01x02_Pin") (at 114 67 0) (unit 1) (exclude_from_sim no) (in_bom yes) (on_board yes) (dnp no)
     (property "Reference" "J1" (at 114 59.38 0) (effects (font (size 1.27 1.27))))
@@
     (property "Footprint" "!fablabs-kicad-library:TerminalBlock_Phoenix_MKDS-1,5-2-5.08_1x02_P5.08mm_Horizontal" (at 114 77.16 0) (effects (font (size 1.27 1.27)) hide))
     (property "Datasheet" "" (at 114 79.7 0) (effects (font (size 1.27 1.27)) hide))
+    (instances
+      (project "fablabs"
+        (path "/0ffc1615-9aac-459a-a1ce-f9c7f1ed2a31"
+          (reference "J1") (unit 1)
+        )
+      )
+    )
   )
   (label "VIN_1" (at 119.08 67 0) (fields_autoplaced) (effects (font (size 1.27 1.27)) (justify left bottom)))
-  (label "VIN_2" (at 119.08 64.46 0) (fields_autoplaced) (effects (font (size 1.27 1.27)) (justify left bottom)))
+  (label "VIN_2" (at 119.08 69.54 0) (fields_autoplaced) (effects (font (size 1.27 1.27)) (justify left bottom)))
   (symbol (lib_id "!fablabs-kicad-library:Conn_01x02_Pin") (at 30 99 0) (unit 1) (exclude_from_sim no) (in_bom yes) (on_board yes) (dnp no)
     (property "Reference" "J2" (at 30 91.38 0) (effects (font (size 1.27 1.27))))
@@
     (property "Footprint" "!fablabs-kicad-library:TerminalBlock_Phoenix_MKDS-1,5-2-5.08_1x02_P5.08mm_Horizontal" (at 30 109.16 0) (effects (font (size 1.27 1.27)) hide))
     (property "Datasheet" "" (at 30 111.7 0) (effects (font (size 1.27 1.27)) hide))
+    (instances
+      (project "fablabs"
+        (path "/719f443c-f026-4cc7-8c65-9721d1c6d9dd"
+          (reference "J2") (unit 1)
+        )
+      )
+    )
   )
   (label "5V_OUT_1" (at 35.08 99 0) (fields_autoplaced) (effects (font (size 1.27 1.27)) (justify left bottom)))
-  (label "5V_OUT_2" (at 35.08 96.46 0) (fields_autoplaced) (effects (font (size 1.27 1.27)) (justify left bottom)))
+  (label "5V_OUT_2" (at 35.08 101.54 0) (fields_autoplaced) (effects (font (size 1.27 1.27)) (justify left bottom)))
+  (sheet_instances
+    (path "/" (page "1"))
+  )
 )
