File: !fablabs-kicad-library.kicad_blocks/POWER_LDO_ADJUSTABLE_GENERIC_SOT223.kicad_block/POWER_LDO_ADJUSTABLE_GENERIC_SOT223.kicad_pcb (KiCad board)
At the start: 2 copper layers, 7 parts, among them J1 VIN, J2 VOUT, U1 LM1117-ADJ

Commit message: Fixed some bugs
Parts:
- moved C2 177.2 mm to (170.0, 50.0)
- moved C1 148.7 mm to (140.0, 50.0)
- moved R2 120.8 mm to (110.0, 50.0)
- moved J2 113.1 mm to (80.0, 80.0)
- moved J1 94.3 mm to (50.0, 80.0)
- moved R1 94.3 mm to (80.0, 50.0)
- moved U1 70.7 mm to (50.0, 50.0)
Changed lines of the file:
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@@
-(kicad_pcb (version 20240108) (generator "fablabs-kicad-library-builder") (generator_version "1.0.0")
+(kicad_pcb (version 20260206) (generator "eeschema") (generator_version "10.0")
   (general (thickness 1.6))
   (paper "A4")
@@
   	(generator_version "10.0")
   	(layer "F.Cu")
+    (at 50 50 0)
   	(descr "module CMS SOT223 4 pins")
   	(tags "CMS SOT")
   	(property "Reference" "U1"
-    (at 50 50 0)
+  		(at 0 -4.5 0)
   		(layer "F.SilkS")
   		(effects
@@
   	)
   	(embedded_fonts no)
-  	(model "${KICAD10_3DMODEL_DIR}/Package_TO_SOT_SMD.3dshapes/SOT-223.step"
+  	(model "${KIPRJMOD}/libs/!fablabs-kicad-library.3dshapes/SOT-223.step"
   		(offset
   			(xyz 0 0 0)
@@
   	(generator "kicad-footprint-generator")
   	(layer "F.Cu")
+    (at 80 50 0)
   	(descr "Resistor SMD 0603 (1608 Metric), square (rectangular) end terminal, IPC-7351 nominal, (Body size source: IPC-SM-782 page 72, https://www.pcb-3d.com/wordpress/wp-content/uploads/ipc-sm-782a_amendment_1_and_2.pdf)")
   	(tags "resistor")
   	(property "Reference" "R1"
-    (at 80 50 0)
+  		(at 0 -1.43 0)
   		(layer "F.SilkS")
   		(effects
@@
   	)
   	(embedded_fonts no)
-  	(model "${KICAD10_3DMODEL_DIR}/Resistor_SMD.3dshapes/R_0603_1608Metric.step"
+  	(model "${KIPRJMOD}/libs/!fablabs-kicad-library.3dshapes/R_0603_1608Metric.step"
   		(offset
   			(xyz 0 0 0)
@@
   	(generator "kicad-footprint-generator")
   	(layer "F.Cu")
+    (at 110 50 0)
   	(descr "Resistor SMD 0603 (1608 Metric), square (rectangular) end terminal, IPC-7351 nominal, (Body size source: IPC-SM-782 page 72, https://www.pcb-3d.com/wordpress/wp-content/uploads/ipc-sm-782a_amendment_1_and_2.pdf)")
   	(tags "resistor")
   	(property "Reference" "R2"
-    (at 110 50 0)
+  		(at 0 -1.43 0)
   		(layer "F.SilkS")
   		(effects
@@
   	)
   	(embedded_fonts no)
-  	(model "${KICAD10_3DMODEL_DIR}/Resistor_SMD.3dshapes/R_0603_1608Metric.step"
+  	(model "${KIPRJMOD}/libs/!fablabs-kicad-library.3dshapes/R_0603_1608Metric.step"
   		(offset
   			(xyz 0 0 0)
@@
   	(generator "kicad-footprint-generator")
   	(layer "F.Cu")
+    (at 140 50 0)
   	(descr "Capacitor SMD 0805 (2012 Metric), square (rectangular) end terminal, IPC-7351 nominal, (Body size source: IPC-SM-782 page 76, https://www.pcb-3d.com/wordpress/wp-content/uploads/ipc-sm-782a_amendment_1_and_2.pdf, https://docs.google.com/spreadsheets/d/1BsfQQcO9C6DZCsRaXUlFlo91Tg2WpOkGARC1WS5S8t0/edit?usp=sharing)")
   	(tags "capacitor")
   	(property "Reference" "C1"
-    (at 140 50 0)
+  		(at 0 -1.68 0)
   		(layer "F.SilkS")
   		(effects
@@
   	(generator "kicad-footprint-generator")
   	(layer "F.Cu")
+    (at 170 50 0)
   	(descr "Capacitor SMD 0805 (2012 Metric), square (rectangular) end terminal, IPC-7351 nominal, (Body size source: IPC-SM-782 page 76, https://www.pcb-3d.com/wordpress/wp-content/uploads/ipc-sm-782a_amendment_1_and_2.pdf, https://docs.google.com/spreadsheets/d/1BsfQQcO9C6DZCsRaXUlFlo91Tg2WpOkGARC1WS5S8t0/edit?usp=sharing)")
   	(tags "capacitor")
   	(property "Reference" "C2"
-    (at 170 50 0)
+  		(at 0 -1.68 0)
   		(layer "F.SilkS")
   		(effects
@@
   	(generator "kicad-footprint-generator")
   	(layer "F.Cu")
+    (at 50 80 0)
   	(descr "Through hole straight pin header, 1x02, 2.54mm pitch, single row")
   	(tags "Through hole pin header THT 1x02 2.54mm single row")
   	(property "Reference" "J1"
-    (at 50 80 0)
+  		(at 0 -2.38 0)
   		(layer "F.SilkS")
   		(effects
@@
   	(generator "kicad-footprint-generator")
   	(layer "F.Cu")
+    (at 80 80 0)
   	(descr "Through hole straight pin header, 1x02, 2.54mm pitch, single row")
   	(tags "Through hole pin header THT 1x02 2.54mm single row")
   	(property "Reference" "J2"
-    (at 80 80 0)
-  		(layer "F.SilkS")
-  		(effects
+  		(at 0 -2.38 0)
+  		(layer "F.SilkS")
+  		(effects
