File: !fablabs-kicad-library.kicad_blocks/POWER_LOAD_SWITCH_GENERIC.kicad_block/POWER_LOAD_SWITCH_GENERIC.kicad_sch (KiCad schematic)
At the start: 5 parts, among them J1 LOAD_SWITCH_IO, Q1 PMOS_LOAD_SWITCH

Commit message: Fixed some bugs
Connections:
- net EN: now also R2.1
- net GATE: now also C1.1, Q1.1 (G), R1.1, R2.2
- net LOAD_SW_1: now also J1.1 (Pin_1)
- net LOAD_SW_2: now also J1.2 (Pin_2)
- net LOAD_SW_3: now also J1.3 (Pin_3)
- net VIN: now also C1.2, Q1.2 (S), R1.2
- net VSW: now also Q1.3 (D)
Changed lines of the file:
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@@
-(kicad_sch (version 20250114) (generator "fablabs-kicad-library-builder") (generator_version "1.0.0")
+(kicad_sch (version 20260306) (generator "eeschema") (generator_version "10.0")
   (paper "A4")
   (title_block
@@
     (property "Footprint" "!fablabs-kicad-library:SOT-23" (at 30 45.16 0) (effects (font (size 1.27 1.27)) hide))
     (property "Datasheet" "" (at 30 47.7 0) (effects (font (size 1.27 1.27)) hide))
+    (instances
+      (project "fablabs"
+        (path "/6c54ec89-d7f3-41ab-80de-db9522721394"
+          (reference "Q1") (unit 1)
+        )
+      )
+    )
   )
   (label "GATE" (at 24.92 35 0) (fields_autoplaced) (effects (font (size 1.27 1.27)) (justify left bottom)))
-  (label "VIN" (at 32.54 29.92 0) (fields_autoplaced) (effects (font (size 1.27 1.27)) (justify left bottom)))
-  (label "VSW" (at 32.54 40.08 0) (fields_autoplaced) (effects (font (size 1.27 1.27)) (justify left bottom)))
+  (label "VIN" (at 32.54 40.08 0) (fields_autoplaced) (effects (font (size 1.27 1.27)) (justify left bottom)))
+  (label "VSW" (at 32.54 29.92 0) (fields_autoplaced) (effects (font (size 1.27 1.27)) (justify left bottom)))
   (symbol (lib_id "!fablabs-kicad-library:R") (at 72 35 0) (unit 1) (exclude_from_sim no) (in_bom yes) (on_board yes) (dnp no)
     (property "Reference" "R1" (at 72 27.38 0) (effects (font (size 1.27 1.27))))
@@
     (property "Footprint" "!fablabs-kicad-library:R_0603_1608Metric" (at 72 45.16 0) (effects (font (size 1.27 1.27)) hide))
     (property "Datasheet" "" (at 72 47.7 0) (effects (font (size 1.27 1.27)) hide))
+    (instances
+      (project "fablabs"
+        (path "/fade73eb-787c-4efc-9dc8-a86592d84d7a"
+          (reference "R1") (unit 1)
+        )
+      )
+    )
   )
-  (label "GATE" (at 72 38.81 0) (fields_autoplaced) (effects (font (size 1.27 1.27)) (justify left bottom)))
-  (label "VIN" (at 72 31.19 0) (fields_autoplaced) (effects (font (size 1.27 1.27)) (justify left bottom)))
+  (label "GATE" (at 72 31.19 0) (fields_autoplaced) (effects (font (size 1.27 1.27)) (justify left bottom)))
+  (label "VIN" (at 72 38.81 0) (fields_autoplaced) (effects (font (size 1.27 1.27)) (justify left bottom)))
   (symbol (lib_id "!fablabs-kicad-library:R") (at 114 35 0) (unit 1) (exclude_from_sim no) (in_bom yes) (on_board yes) (dnp no)
     (property "Reference" "R2" (at 114 27.38 0) (effects (font (size 1.27 1.27))))
@@
     (property "Footprint" "!fablabs-kicad-library:R_0603_1608Metric" (at 114 45.16 0) (effects (font (size 1.27 1.27)) hide))
     (property "Datasheet" "" (at 114 47.7 0) (effects (font (size 1.27 1.27)) hide))
+    (instances
+      (project "fablabs"
+        (path "/caa98093-5722-412f-b9e8-f29f558d3a8a"
+          (reference "R2") (unit 1)
+        )
+      )
+    )
   )
-  (label "EN" (at 114 38.81 0) (fields_autoplaced) (effects (font (size 1.27 1.27)) (justify left bottom)))
-  (label "GATE" (at 114 31.19 0) (fields_autoplaced) (effects (font (size 1.27 1.27)) (justify left bottom)))
+  (label "EN" (at 114 31.19 0) (fields_autoplaced) (effects (font (size 1.27 1.27)) (justify left bottom)))
+  (label "GATE" (at 114 38.81 0) (fields_autoplaced) (effects (font (size 1.27 1.27)) (justify left bottom)))
   (symbol (lib_id "!fablabs-kicad-library:C") (at 30 67 0) (unit 1) (exclude_from_sim no) (in_bom yes) (on_board yes) (dnp no)
     (property "Reference" "C1" (at 30 59.38 0) (effects (font (size 1.27 1.27))))
@@
     (property "Footprint" "!fablabs-kicad-library:C_0603_1608Metric" (at 30 77.16 0) (effects (font (size 1.27 1.27)) hide))
     (property "Datasheet" "" (at 30 79.7 0) (effects (font (size 1.27 1.27)) hide))
+    (instances
+      (project "fablabs"
+        (path "/7be32c9e-2f79-4ef8-a689-91e7ded457ad"
+          (reference "C1") (unit 1)
+        )
+      )
+    )
   )
-  (label "GATE" (at 30 70.81 0) (fields_autoplaced) (effects (font (size 1.27 1.27)) (justify left bottom)))
-  (label "VIN" (at 30 63.19 0) (fields_autoplaced) (effects (font (size 1.27 1.27)) (justify left bottom)))
+  (label "GATE" (at 30 63.19 0) (fields_autoplaced) (effects (font (size 1.27 1.27)) (justify left bottom)))
+  (label "VIN" (at 30 70.81 0) (fields_autoplaced) (effects (font (size 1.27 1.27)) (justify left bottom)))
   (symbol (lib_id "!fablabs-kicad-library:Conn_01x03_Pin") (at 72 67 0) (unit 1) (exclude_from_sim no) (in_bom yes) (on_board yes) (dnp no)
     (property "Reference" "J1" (at 72 59.38 0) (effects (font (size 1.27 1.27))))
@@
     (property "Footprint" "!fablabs-kicad-library:PinHeader_1x03_P2.54mm_Vertical" (at 72 77.16 0) (effects (font (size 1.27 1.27)) hide))
     (property "Datasheet" "" (at 72 79.7 0) (effects (font (size 1.27 1.27)) hide))
+    (instances
+      (project "fablabs"
+        (path "/21660a17-e653-427e-bf83-3ddcaca211ad"
+          (reference "J1") (unit 1)
+        )
+      )
+    )
   )
-  (label "LOAD_SW_1" (at 77.08 69.54 0) (fields_autoplaced) (effects (font (size 1.27 1.27)) (justify left bottom)))
+  (label "LOAD_SW_1" (at 77.08 64.46 0) (fields_autoplaced) (effects (font (size 1.27 1.27)) (justify left bottom)))
   (label "LOAD_SW_2" (at 77.08 67 0) (fields_autoplaced) (effects (font (size 1.27 1.27)) (justify left bottom)))
-  (label "LOAD_SW_3" (at 77.08 64.46 0) (fields_autoplaced) (effects (font (size 1.27 1.27)) (justify left bottom)))
+  (label "LOAD_SW_3" (at 77.08 69.54 0) (fields_autoplaced) (effects (font (size 1.27 1.27)) (justify left bottom)))
+  (sheet_instances
+    (path "/" (page "1"))
+  )
 )
