File: !fablabs-kicad-library.kicad_blocks/PROTECTION_INPUT_TVS_FUSE_REVERSE_DIODE.kicad_block/PROTECTION_INPUT_TVS_FUSE_REVERSE_DIODE.kicad_pcb (KiCad board)
At the start: 2 copper layers, 6 parts, among them J1 IN, J2 OUT

Commit message: Fixed some bugs
Parts:
- moved J1 177.2 mm to (170.0, 50.0)
- moved C1 148.7 mm to (140.0, 50.0)
- moved D2 120.8 mm to (110.0, 50.0)
- moved D1 94.3 mm to (80.0, 50.0)
- moved J2 94.3 mm to (50.0, 80.0)
- moved F1 70.7 mm to (50.0, 50.0)
Changed lines of the file:
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@@
-(kicad_pcb (version 20240108) (generator "fablabs-kicad-library-builder") (generator_version "1.0.0")
+(kicad_pcb (version 20260206) (generator "eeschema") (generator_version "10.0")
   (general (thickness 1.6))
   (paper "A4")
@@
   	(generator "kicad-footprint-generator")
   	(layer "F.Cu")
+    (at 50 50 0)
   	(descr "Fuse SMD 1206 (3216 Metric), square (rectangular) end terminal, IPC-7351 nominal, (Body size source: http://www.tortai-tech.com/upload/download/2011102023233369053.pdf)")
   	(tags "fuse")
   	(property "Reference" "F1"
-    (at 50 50 0)
+  		(at 0 -1.83 0)
   		(layer "F.SilkS")
   		(effects
@@
   	(generator_version "10.0")
   	(layer "F.Cu")
+    (at 80 50 0)
   	(descr "SOD-123")
   	(tags "SOD-123")
   	(property "Reference" "D1"
-    (at 80 50 0)
+  		(at 0 -2 0)
   		(layer "F.SilkS")
   		(effects
@@
   	(generator_version "10.0")
   	(layer "F.Cu")
+    (at 110 50 0)
   	(descr "SOD-123")
   	(tags "SOD-123")
   	(property "Reference" "D2"
-    (at 110 50 0)
+  		(at 0 -2 0)
   		(layer "F.SilkS")
   		(effects
@@
   	(generator "kicad-footprint-generator")
   	(layer "F.Cu")
+    (at 140 50 0)
   	(descr "Capacitor SMD 0805 (2012 Metric), square (rectangular) end terminal, IPC-7351 nominal, (Body size source: IPC-SM-782 page 76, https://www.pcb-3d.com/wordpress/wp-content/uploads/ipc-sm-782a_amendment_1_and_2.pdf, https://docs.google.com/spreadsheets/d/1BsfQQcO9C6DZCsRaXUlFlo91Tg2WpOkGARC1WS5S8t0/edit?usp=sharing)")
   	(tags "capacitor")
   	(property "Reference" "C1"
-    (at 140 50 0)
+  		(at 0 -1.68 0)
   		(layer "F.SilkS")
   		(effects
@@
   	(generator "kicad-footprint-generator")
   	(layer "F.Cu")
+    (at 170 50 0)
   	(descr "Through hole straight pin header, 1x02, 2.54mm pitch, single row")
   	(tags "Through hole pin header THT 1x02 2.54mm single row")
   	(property "Reference" "J1"
-    (at 170 50 0)
+  		(at 0 -2.38 0)
   		(layer "F.SilkS")
   		(effects
@@
   	(generator "kicad-footprint-generator")
   	(layer "F.Cu")
+    (at 50 80 0)
   	(descr "Through hole straight pin header, 1x02, 2.54mm pitch, single row")
   	(tags "Through hole pin header THT 1x02 2.54mm single row")
   	(property "Reference" "J2"
-    (at 50 80 0)
-  		(layer "F.SilkS")
-  		(effects
+  		(at 0 -2.38 0)
+  		(layer "F.SilkS")
+  		(effects
