File: !fablabs-kicad-library.kicad_blocks/PROTOCOL_AVR_ISP_6PIN.kicad_block/PROTOCOL_AVR_ISP_6PIN.kicad_pcb (KiCad board)
At the start: 2 copper layers, 1 part, among them J1 AVR_ISP_6

Commit message: Fixed some bugs
Parts:
- moved J1 70.7 mm to (50.0, 50.0)
Changed lines of the file:
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@@
-(kicad_pcb (version 20240108) (generator "fablabs-kicad-library-builder") (generator_version "1.0.0")
+(kicad_pcb (version 20260206) (generator "eeschema") (generator_version "10.0")
   (general (thickness 1.6))
   (paper "A4")
@@
   	(generator "kicad-footprint-generator")
   	(layer "F.Cu")
+    (at 50 50 0)
   	(descr "Through hole straight pin header, 2x03, 2.54mm pitch, double rows")
   	(tags "Through hole pin header THT 2x03 2.54mm double row")
   	(property "Reference" "J1"
-    (at 50 50 0)
+  		(at 1.27 -2.38 0)
   		(layer "F.SilkS")
   		(effects
