File: !fablabs-kicad-library.kicad_blocks/PROTOCOL_SPI_SENSOR_PORT.kicad_block/PROTOCOL_SPI_SENSOR_PORT.kicad_pcb (KiCad board)
At the start: 2 copper layers, 2 parts, among them J1 SPI_SENSOR

Commit message: Fixed some bugs
Parts:
- moved C1 94.3 mm to (80.0, 50.0)
- moved J1 70.7 mm to (50.0, 50.0)
Changed lines of the file:
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@@
-(kicad_pcb (version 20240108) (generator "fablabs-kicad-library-builder") (generator_version "1.0.0")
+(kicad_pcb (version 20260206) (generator "eeschema") (generator_version "10.0")
   (general (thickness 1.6))
   (paper "A4")
@@
   	(generator "kicad-footprint-generator")
   	(layer "F.Cu")
+    (at 50 50 0)
   	(descr "Through hole straight pin header, 1x08, 2.54mm pitch, single row")
   	(tags "Through hole pin header THT 1x08 2.54mm single row")
   	(property "Reference" "J1"
-    (at 50 50 0)
+  		(at 0 -2.38 0)
   		(layer "F.SilkS")
   		(effects
@@
   	(generator "kicad-footprint-generator")
   	(layer "F.Cu")
+    (at 80 50 0)
   	(descr "Capacitor SMD 0603 (1608 Metric), square (rectangular) end terminal, IPC-7351 nominal, (Body size source: IPC-SM-782 page 76, https://www.pcb-3d.com/wordpress/wp-content/uploads/ipc-sm-782a_amendment_1_and_2.pdf)")
   	(tags "capacitor")
   	(property "Reference" "C1"
-    (at 80 50 0)
-  		(layer "F.SilkS")
-  		(effects
+  		(at 0 -1.43 0)
+  		(layer "F.SilkS")
+  		(effects
