File: !fablabs-kicad-library.kicad_blocks/PROTOCOL_SWD_10PIN_ARM_HEADER.kicad_block/PROTOCOL_SWD_10PIN_ARM_HEADER.kicad_sch (KiCad schematic)
At the start: 1 part, among them J1 ARM_SWD_10

Commit message: Fixed some bugs
Connections:
- net GND: now also J1.3 (Pin_3), J1.5 (Pin_5), J1.9 (Pin_9)
- net NC: now also J1.7 (Pin_7), J1.8 (Pin_8)
- net NRST: now also J1.10 (Pin_10)
- net SWCLK: now also J1.4 (Pin_4)
- net SWDIO: now also J1.2 (Pin_2)
- net SWO: now also J1.6 (Pin_6)
- net VTREF: now also J1.1 (Pin_1)
Changed lines of the file:
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@@
-(kicad_sch (version 20250114) (generator "fablabs-kicad-library-builder") (generator_version "1.0.0")
+(kicad_sch (version 20260306) (generator "eeschema") (generator_version "10.0")
   (paper "A4")
   (title_block
@@
     (property "Footprint" "!fablabs-kicad-library:PinHeader_2x05_P1.27mm_Vertical" (at 30 45.16 0) (effects (font (size 1.27 1.27)) hide))
     (property "Datasheet" "" (at 30 47.7 0) (effects (font (size 1.27 1.27)) hide))
+    (instances
+      (project "fablabs"
+        (path "/b9315d73-0c9b-4f4c-8639-b27c5274eb59"
+          (reference "J1") (unit 1)
+        )
+      )
+    )
   )
-  (label "VTREF" (at 24.92 40.08 0) (fields_autoplaced) (effects (font (size 1.27 1.27)) (justify left bottom)))
-  (label "SWDIO" (at 37.62 40.08 0) (fields_autoplaced) (effects (font (size 1.27 1.27)) (justify left bottom)))
-  (label "GND" (at 24.92 37.54 0) (fields_autoplaced) (effects (font (size 1.27 1.27)) (justify left bottom)))
-  (label "SWCLK" (at 37.62 37.54 0) (fields_autoplaced) (effects (font (size 1.27 1.27)) (justify left bottom)))
+  (label "VTREF" (at 24.92 29.92 0) (fields_autoplaced) (effects (font (size 1.27 1.27)) (justify left bottom)))
+  (label "SWDIO" (at 37.62 29.92 0) (fields_autoplaced) (effects (font (size 1.27 1.27)) (justify left bottom)))
+  (label "GND" (at 24.92 32.46 0) (fields_autoplaced) (effects (font (size 1.27 1.27)) (justify left bottom)))
+  (label "SWCLK" (at 37.62 32.46 0) (fields_autoplaced) (effects (font (size 1.27 1.27)) (justify left bottom)))
   (label "GND" (at 24.92 35 0) (fields_autoplaced) (effects (font (size 1.27 1.27)) (justify left bottom)))
   (label "SWO" (at 37.62 35 0) (fields_autoplaced) (effects (font (size 1.27 1.27)) (justify left bottom)))
-  (label "NC" (at 24.92 32.46 0) (fields_autoplaced) (effects (font (size 1.27 1.27)) (justify left bottom)))
-  (label "NC" (at 37.62 32.46 0) (fields_autoplaced) (effects (font (size 1.27 1.27)) (justify left bottom)))
-  (label "GND" (at 24.92 29.92 0) (fields_autoplaced) (effects (font (size 1.27 1.27)) (justify left bottom)))
-  (label "NRST" (at 37.62 29.92 0) (fields_autoplaced) (effects (font (size 1.27 1.27)) (justify left bottom)))
+  (label "NC" (at 24.92 37.54 0) (fields_autoplaced) (effects (font (size 1.27 1.27)) (justify left bottom)))
+  (label "NC" (at 37.62 37.54 0) (fields_autoplaced) (effects (font (size 1.27 1.27)) (justify left bottom)))
+  (label "GND" (at 24.92 40.08 0) (fields_autoplaced) (effects (font (size 1.27 1.27)) (justify left bottom)))
+  (label "NRST" (at 37.62 40.08 0) (fields_autoplaced) (effects (font (size 1.27 1.27)) (justify left bottom)))
+  (sheet_instances
+    (path "/" (page "1"))
+  )
 )
