File: !fablabs-kicad-library.kicad_blocks/RF_GNSS_NEO_M8N_MODULE.kicad_block/RF_GNSS_NEO_M8N_MODULE.kicad_pcb (KiCad board)
At the start: 2 copper layers, 5 parts, among them J1 U.FL, J2 GNSS_UART, U1 NEO-M8N

Commit message: Fixed some bugs
Parts:
- moved J2 177.2 mm to (170.0, 50.0)
- moved J1 148.7 mm to (140.0, 50.0)
- moved C2 120.8 mm to (110.0, 50.0)
- moved C1 94.3 mm to (80.0, 50.0)
- moved U1 70.7 mm to (50.0, 50.0)
Changed lines of the file:
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@@
-(kicad_pcb (version 20240108) (generator "fablabs-kicad-library-builder") (generator_version "1.0.0")
+(kicad_pcb (version 20260206) (generator "eeschema") (generator_version "10.0")
   (general (thickness 1.6))
   (paper "A4")
@@
   	(generator_version "10.0")
   	(layer "F.Cu")
+    (at 50 50 0)
   	(descr "ublox NEO 6/7/8, (https://www.u-blox.com/sites/default/files/NEO-8Q-NEO-M8-FW3_HardwareIntegrationManual_%28UBX-15029985%29_0.pdf)")
   	(tags "GPS ublox NEO 6/7/8")
   	(property "Reference" "U1"
-    (at 50 50 0)
+  		(at 0 -9 0)
   		(layer "F.SilkS")
   		(effects
@@
   	(generator "kicad-footprint-generator")
   	(layer "F.Cu")
+    (at 80 50 0)
   	(descr "Capacitor SMD 0603 (1608 Metric), square (rectangular) end terminal, IPC-7351 nominal, (Body size source: IPC-SM-782 page 76, https://www.pcb-3d.com/wordpress/wp-content/uploads/ipc-sm-782a_amendment_1_and_2.pdf)")
   	(tags "capacitor")
   	(property "Reference" "C1"
-    (at 80 50 0)
+  		(at 0 -1.43 0)
   		(layer "F.SilkS")
   		(effects
@@
   	(generator "kicad-footprint-generator")
   	(layer "F.Cu")
+    (at 110 50 0)
   	(descr "Capacitor SMD 0805 (2012 Metric), square (rectangular) end terminal, IPC-7351 nominal, (Body size source: IPC-SM-782 page 76, https://www.pcb-3d.com/wordpress/wp-content/uploads/ipc-sm-782a_amendment_1_and_2.pdf, https://docs.google.com/spreadsheets/d/1BsfQQcO9C6DZCsRaXUlFlo91Tg2WpOkGARC1WS5S8t0/edit?usp=sharing)")
   	(tags "capacitor")
   	(property "Reference" "C2"
-    (at 110 50 0)
+  		(at 0 -1.68 0)
   		(layer "F.SilkS")
   		(effects
@@
   	(generator_version "10.0")
   	(layer "F.Cu")
+    (at 140 50 0)
   	(descr "Hirose U.FL Coaxial (https://www.hirose.com/en/product/document?clcode=CL0331-0472-2-01&productname=U.FL-R-SMT-1(01)&series=U.FL&documenttype=2DDrawing&lang=en&documentid=0000940668)")
   	(tags "Hirose U.FL Coaxial")
   	(property "Reference" "J1"
-    (at 140 50 0)
+  		(at 0 -3.2 0)
   		(layer "F.SilkS")
   		(effects
@@
   	(generator "kicad-footprint-generator")
   	(layer "F.Cu")
+    (at 170 50 0)
   	(descr "Through hole straight pin header, 1x06, 2.54mm pitch, single row")
   	(tags "Through hole pin header THT 1x06 2.54mm single row")
   	(property "Reference" "J2"
-    (at 170 50 0)
-  		(layer "F.SilkS")
-  		(effects
+  		(at 0 -2.38 0)
+  		(layer "F.SilkS")
+  		(effects
