File: !fablabs-kicad-library.kicad_blocks/SENSOR_DS18B20_ONEWIRE_LOCAL.kicad_block/SENSOR_DS18B20_ONEWIRE_LOCAL.kicad_sch (KiCad schematic)
At the start: 4 parts, among them J1 ONEWIRE_EXT, U1 DS18B20

Commit message: Fixed some bugs
Connections:
- net DQ: now also R1.1
- net GND: now also C1.2
- net OW_EXT_1: now also J1.1 (Pin_1)
- net OW_EXT_2: now also J1.2 (Pin_2)
- net OW_EXT_3: now also J1.3 (Pin_3)
- net VDD: now also C1.1, R1.2
Changed lines of the file:
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@@
-(kicad_sch (version 20250114) (generator "fablabs-kicad-library-builder") (generator_version "1.0.0")
+(kicad_sch (version 20260306) (generator "eeschema") (generator_version "10.0")
   (paper "A4")
   (title_block
@@
     (property "MPN" "DS18B20+" (at 30 50.24 0) (effects (font (size 1.27 1.27)) hide))
     (property "Manufacturer" "Analog Devices/Maxim" (at 30 52.78 0) (effects (font (size 1.27 1.27)) hide))
+    (instances
+      (project "fablabs"
+        (path "/f8f5e014-6697-4cd5-89b1-c34dcfe038ae"
+          (reference "U1") (unit 1)
+        )
+      )
+    )
   )
   (symbol (lib_id "!fablabs-kicad-library:R") (at 72 35 0) (unit 1) (exclude_from_sim no) (in_bom yes) (on_board yes) (dnp no)
@@
     (property "Footprint" "!fablabs-kicad-library:R_0603_1608Metric" (at 72 45.16 0) (effects (font (size 1.27 1.27)) hide))
     (property "Datasheet" "" (at 72 47.7 0) (effects (font (size 1.27 1.27)) hide))
+    (instances
+      (project "fablabs"
+        (path "/cb4157bc-54d7-4cbf-88b4-db8e1a6b16a6"
+          (reference "R1") (unit 1)
+        )
+      )
+    )
   )
-  (label "DQ" (at 72 38.81 0) (fields_autoplaced) (effects (font (size 1.27 1.27)) (justify left bottom)))
-  (label "VDD" (at 72 31.19 0) (fields_autoplaced) (effects (font (size 1.27 1.27)) (justify left bottom)))
+  (label "DQ" (at 72 31.19 0) (fields_autoplaced) (effects (font (size 1.27 1.27)) (justify left bottom)))
+  (label "VDD" (at 72 38.81 0) (fields_autoplaced) (effects (font (size 1.27 1.27)) (justify left bottom)))
   (symbol (lib_id "!fablabs-kicad-library:C") (at 114 35 0) (unit 1) (exclude_from_sim no) (in_bom yes) (on_board yes) (dnp no)
     (property "Reference" "C1" (at 114 27.38 0) (effects (font (size 1.27 1.27))))
@@
     (property "Footprint" "!fablabs-kicad-library:C_0603_1608Metric" (at 114 45.16 0) (effects (font (size 1.27 1.27)) hide))
     (property "Datasheet" "" (at 114 47.7 0) (effects (font (size 1.27 1.27)) hide))
+    (instances
+      (project "fablabs"
+        (path "/f9406474-d354-4984-82b8-a787d18d5b47"
+          (reference "C1") (unit 1)
+        )
+      )
+    )
   )
-  (label "VDD" (at 114 38.81 0) (fields_autoplaced) (effects (font (size 1.27 1.27)) (justify left bottom)))
-  (label "GND" (at 114 31.19 0) (fields_autoplaced) (effects (font (size 1.27 1.27)) (justify left bottom)))
+  (label "VDD" (at 114 31.19 0) (fields_autoplaced) (effects (font (size 1.27 1.27)) (justify left bottom)))
+  (label "GND" (at 114 38.81 0) (fields_autoplaced) (effects (font (size 1.27 1.27)) (justify left bottom)))
   (symbol (lib_id "!fablabs-kicad-library:Conn_01x03_Pin") (at 30 67 0) (unit 1) (exclude_from_sim no) (in_bom yes) (on_board yes) (dnp no)
     (property "Reference" "J1" (at 30 59.38 0) (effects (font (size 1.27 1.27))))
@@
     (property "Footprint" "!fablabs-kicad-library:PinHeader_1x03_P2.54mm_Vertical" (at 30 77.16 0) (effects (font (size 1.27 1.27)) hide))
     (property "Datasheet" "" (at 30 79.7 0) (effects (font (size 1.27 1.27)) hide))
+    (instances
+      (project "fablabs"
+        (path "/fa88fc2c-0fcf-4ad3-98b2-cf28c2d1a591"
+          (reference "J1") (unit 1)
+        )
+      )
+    )
   )
-  (label "OW_EXT_1" (at 35.08 69.54 0) (fields_autoplaced) (effects (font (size 1.27 1.27)) (justify left bottom)))
+  (label "OW_EXT_1" (at 35.08 64.46 0) (fields_autoplaced) (effects (font (size 1.27 1.27)) (justify left bottom)))
   (label "OW_EXT_2" (at 35.08 67 0) (fields_autoplaced) (effects (font (size 1.27 1.27)) (justify left bottom)))
-  (label "OW_EXT_3" (at 35.08 64.46 0) (fields_autoplaced) (effects (font (size 1.27 1.27)) (justify left bottom)))
+  (label "OW_EXT_3" (at 35.08 69.54 0) (fields_autoplaced) (effects (font (size 1.27 1.27)) (justify left bottom)))
+  (sheet_instances
+    (path "/" (page "1"))
+  )
 )
